File: kicad/ta-expt-v2.kicad_sch (KiCad schematic)
At the start: 46 parts, among them IC1 STS5PF30L, IC2 IS25LP128F-JBLA3, IC3 STM32L496VGT3, J1 Conn_01x16, J2 Conn_01x16, J3 Conn_01x04, J4 Conn_01x04, J5 Conn_01x05, J6 Conn_01x05, J7 Conn_01x04, J8 Conn_02x06_Odd_Even, J9 USB_C_Receptacle_USB2.0, U1 TPS7A0533PDBV, Y1 ABS07AIG-32.768kHz-T, Y3 ABM8AIG-16.000MHZ-12-2Z-T

Commit message: Add files via upload
Parts:
- removed D1, D2: BAR42FILM, Package_TO_SOT_SMD:SOT-23, symbol Diode:BAR42FILM
- added IC4: BAR43SFILM, ta-expt-v2-100:SOTFL50P160X78-3N, symbol BAR43SFILM:BAR43SFILM
- added R3: MCT06030C1002FP500, ta-expt:RESC1608X55N, symbol ta-expt:MCT06030C1002FP500
- added R4: MCT06030C1002FP500, ta-expt-v2-100:RESC1608X55N, symbol ta-expt:MCT06030C1002FP500
- C1, C14, C16, C17, C18, C19, C2, C20, C21, C22, C3, C4, C5, C6, C7, C8, C9: footprint ta-expt:CAPC1608X90N -> ta-expt-v2-100:CAPC1608X90N
- C23: footprint ta-expt:CAPC1608X50N -> ta-expt-v2-100:CAPC1608X50N
- FB1: footprint ta-expt:BEADC1608X95N -> ta-expt-v2-100:BEADC1608X95N
- IC1: footprint SOIC127P600X175-8N -> ta-expt-v2-100:SOIC127P600X175-8N
- IC2: footprint ta-expt:SOIC127P790X216-8N -> ta-expt-v2-100:SOIC127P790X216-8N
- J1, J2: footprint ta-expt:PinSocket_1x16_TartanArtibeus -> ta-expt-v2-100:PinSocket_1x16_TartanArtibeus
- J3, J4: footprint ta-expt:PinSocket_4x1_TartanArtibeus -> ta-expt-v2-100:PinSocket_4x1_TartanArtibeus
- J5, J6: footprint ta-expt:PinSocket_1x5_TartanArtibeus -> ta-expt-v2-100:PinSocket_1x5_TartanArtibeus
- J7: footprint ta-expt:MountingHoles_TartanArtibeus -> ta-expt-v2-100:MountingHoles_TartanArtibeus
- J8: footprint ta-expt:PinSocket_6x2_TartanArtibeus -> ta-expt-v2-100:PinSocket_6x2_TartanArtibeus
- R1, R2, R5, R6, R7, R8, R9: footprint ta-expt:RESC1608X55N -> ta-expt-v2-100:RESC1608X55N
- Y1: footprint ta-expt:ABS07AIG32768kHz71T -> ta-expt-v2-100:ABS07AIG32768kHz71T
- Y3: footprint ta-expt:ABM8AIG25000MHZ122ZT3 -> ta-expt-v2-100:ABM8AIG25000MHZ122ZT3
Connections:
- net VDD_FILT: now also C18.1, C19.2, C20.2, C21.2, C22.2, IC1.1 (S_1), IC1.2 (S_2), IC1.3 (S_3), IC3.100 (VDD_5), IC3.11 (VDD_1), IC3.28 (VDD_2), IC3.50 (VDD_3), IC3.75 (VDD_4); no longer C17.1, U1.5 (OUT)
- net at C15.1: now also IC4.3 (A1/K2)
- net at IC1.4 (G): now also R4.2
- net LDO_OUT: now reaches IC1.5 (D_1), IC1.6 (D_2), IC1.7 (D_3), IC1.8 (D_4)
- net LDO_OUT: now also C17.1, IC3.5 (PE6), U1.5 (OUT), R3.2
- net Control: now reaches IC3.4 (PE5)
- net Control: now also R4.1
- net V_BAT: now reaches IC3.6 (VBAT)
- net V_BAT: now also IC4.1 (A2)
- new net: IC4.2 (K1), R3.1
Other:
- note added: "Replace ====>"
- moved on the sheet: C15
